File: onyks_iot_comm_doordisplay/onyks_iot_comm_doordisplay.kicad_sch (KiCad schematic)
At the start: 43 parts, among them J1 FPC24 (0.5mm), J2 1X6 GOLDPIN, J3 1X2 GOLDPIN, Q1 NMOS, Q2 PMOS, Q4 NPN, Q5 NPN, SW1 SW_Push, SW2 SW_Push, U1 ESP32-WROOM-32D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

Commit message: Added Voltage Divider for Battery Status Measurement
Parts:
- added R10: 100K, symbol Device:R
- added R11: 300K, symbol Device:R
Connections:
- net +BATT: now also R10.1
- net GND: now also R11.2
- net ADC_BATT: now reaches U1.27 (IO16)
- net ADC_BATT: now also R10.2, R11.1
- no-connect marks 25 -> 24
Other:
- note added: "Batt Measure"
- moved on the sheet: C1, C10, C11, C12, C13, C14, C2, C6, C7, C8, C9, J1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

Commit message: fpc footprint, changed diods
Parts:
- C5: footprint (none) -> Capacitor_SMD:C_0805_2012Metric_Pad1.18x1.45mm_HandSolder
- D2, D3, D4: value D -> MBR0530; footprint (none) -> Diode_SMD:D_SOD-123; symbol Device:D -> Diode:MBR0530
- J1: footprint (none) -> Connector_FFC-FPC:TE_2-1734839-4_1x24-1MP_P0.5mm_Horizontal
Changed lines of the file:
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@@
 	)
 	(junction
+		(at 66.04 166.37)
+		(diameter 0)
+		(color 0 0 0 0)
+	)
+	(junction
 		(at 31.75 161.29)
 		(diameter 0)
@@
 	(wire
 		(pts
+			(xy 66.04 166.37) (xy 69.85 166.37)
+		)
+		(stroke
+			(width 0)
+			(type default)
+		)
+	)
+	(wire
+		(pts
 			(xy 45.72 148.59) (xy 45.72 146.05)
 		)
@@
 	(wire
 		(pts
-			(xy 63.5 166.37) (xy 69.85 166.37)
+			(xy 63.5 166.37) (xy 66.04 166.37)
 		)
 		(stroke
@@
 		)
 	)
-	(label "BS"
-		(at 245.11 57.15 0)
-		(fields_autoplaced yes)
-		(effects
-			(font
-				(size 1.27 1.27)
-			)
-			(justify left bottom)
-		)
-	)
 	(label "PREVGL"
 		(at 237.49 95.25 0)
@@
 	)
 	(symbol
-		(lib_id "Device:D")
+		(lib_id "Diode:MBR0530")
 		(at 135.89 147.32 180)
 		(unit 1)
@@
 		(fields_autoplaced yes)
 		(property "Reference" "D2"
-			(at 135.89 140.97 0)
+			(at 136.2075 140.97 0)
 			(effects
 				(font
@@
 			)
 		)
-		(property "Value" "D"
-			(at 135.89 143.51 0)
+		(property "Value" "MBR0530"
+			(at 136.2075 143.51 0)
 			(effects
 				(font
@@
 			)
 		)
-		(property "Footprint" ""
-			(at 135.89 147.32 0)
+		(property "Footprint" "Diode_SMD:D_SOD-123"
+			(at 135.89 142.875 0)
 			(effects
 				(font
@@
 			)
 		)
-		(property "Datasheet" "~"
+		(property "Datasheet" "http://www.mccsemi.com/up_pdf/MBR0520~MBR0580(SOD123).pdf"
 			(at 135.89 147.32 0)
 			(effects
@@
 			)
 		)
-		(property "Description" "Diode"
+		(property "Description" "30V 0.5A Schottky Power Rectifier Diode, SOD-123"
 			(at 135.89 147.32 0)
 			(effects
@@
 	)
 	(symbol
+		(lib_id "power:PWR_FLAG")
+		(at 66.04 166.37 0)
+		(unit 1)
+		(exclude_from_sim no)
+		(in_bom yes)
+		(on_board yes)
+		(dnp no)
+		(fields_autoplaced yes)
+		(property "Reference" "#FLG03"
+			(at 66.04 164.465 0)
+			(effects
+				(font
+					(size 1.27 1.27)
+				)
+				(hide yes)
+			)
+		)
+		(property "Value" "PWR_FLAG"
+			(at 66.04 161.29 0)
+			(effects
+				(font
+					(size 1.27 1.27)
+				)
+			)
+		)
+		(property "Footprint" ""
+			(at 66.04 166.37 0)
+			(effects
+				(font
+					(size 1.27 1.27)
+				)
+				(hide yes)
+			)
+		)
+		(property "Datasheet" "~"
+			(at 66.04 166.37 0)
+			(effects
+				(font
+					(size 1.27 1.27)
+				)
+				(hide yes)
+			)
+		)
+		(property "Description" "Special symbol for telling ERC where power comes from"
+			(at 66.04 166.37 0)
+			(effects
+				(font
+					(size 1.27 1.27)
+				)
+				(hide yes)
+			)
+		)
+		(pin "1"
+		)
+		(instances
+			(project "onyks_iot_comm_doordisplay"
+				(path "/8007192c-fd9f-4325-a65a-9f23d4807586"
+					(reference "#FLG03")
+					(unit 1)
+				)
+			)
+		)
+	)
+	(symbol
 		(lib_id "power:VDD")
 		(at 74.93 166.37 0)
@@
 	)
 	(symbol
-		(lib_id "Device:D")
+		(lib_id "Diode:MBR0530")
 		(at 135.89 133.35 180)
 		(unit 1)
@@
 		(fields_autoplaced yes)
 		(property "Reference" "D4"
-			(at 135.89 127 0)
+			(at 136.2075 127 0)
 			(effects
 				(font
@@
 			)
 		)
-		(property "Value" "D"
-			(at 135.89 129.54 0)
+		(property "Value" "MBR0530"
+			(at 136.2075 129.54 0)
 			(effects
 				(font
@@
 			)
 		)
-		(property "Footprint" ""
-			(at 135.89 133.35 0)
+		(property "Footprint" "Diode_SMD:D_SOD-123"
+			(at 135.89 128.905 0)
 			(effects
 				(font
@@
 			)
 		)
-		(property "Datasheet" "~"
+		(property "Datasheet" "http://www.mccsemi.com/up_pdf/MBR0520~MBR0580(SOD123).pdf"
 			(at 135.89 133.35 0)
 			(effects
@@
 			)
 		)
-		(property "Description" "Diode"
+		(property "Description" "30V 0.5A Schottky Power Rectifier Diode, SOD-123"
 			(at 135.89 133.35 0)
 			(effects
@@
 	)
 	(symbol
-		(lib_id "Device:D")
+		(lib_id "Diode:MBR0530")
 		(at 135.89 124.46 0)
 		(unit 1)
@@
 		(fields_autoplaced yes)
 		(property "Reference" "D3"
-			(at 135.89 118.11 0)
+			(at 135.5725 118.11 0)
 			(effects
 				(font
@@
 			)
 		)
-		(property "Value" "D"
-			(at 135.89 120.65 0)
+		(property "Value" "MBR0530"
+			(at 135.5725 120.65 0)
 			(effects
 				(font
@@
 			)
 		)
-		(property "Footprint" ""
-			(at 135.89 124.46 0)
+		(property "Footprint" "Diode_SMD:D_SOD-123"
+			(at 135.89 128.905 0)
 			(effects
 				(font
@@
 			)
 		)
-		(property "Datasheet" "~"
+		(property "Datasheet" "http://www.mccsemi.com/up_pdf/MBR0520~MBR0580(SOD123).pdf"
 			(at 135.89 124.46 0)
 			(effects
@@
 			)
 		)
-		(property "Description" "Diode"
+		(property "Description" "30V 0.5A Schottky Power Rectifier Diode, SOD-123"
 			(at 135.89 124.46 0)
 			(effects
@@
 			)
 		)
-		(property "Footprint" ""
+		(property "Footprint" "Capacitor_SMD:C_0805_2012Metric_Pad1.18x1.45mm_HandSolder"
 			(at 141.9352 156.21 0)
 			(effects
@@
 			)
 		)
-		(property "Footprint" ""
+		(property "Footprint" "Connector_FFC-FPC:TE_2-1734839-4_1x24-1MP_P0.5mm_Horizontal"
 			(at 259.08 64.77 0)
 			(effects
